Commit message: 自作のxacroに変更

File: summer_robot_description/xacro/robot.xacro (robot description, xacro)
@@ -1,161 +1,254 @@
 <?xml version="1.0"?>
-<robot xmlns:xacro="http://ros.org/wiki/xacro" name="my_omni_robot">
-  <material name="gray">
-    <color rgba="0.8 0.8 0.8 1.0"/>
-  </material>
-  <material name="black">
-    <color rgba="0 0 0 1.0"/>
-  </material>
-  <material name="white">
-    <color rgba="1.0 1.0 1.0 1.0"/>
-  </material>
-  <material name="red">
-    <color rgba="1.0 0 0 1.0"/>
-  </material>
-  <material name="light_red">
-    <color rgba="1.0 0.5 0.5 1.0"/>
-  </material>
-  <material name="yellow">
-    <color rgba="0 1.0 1.0 1.0"/>
-  </material>
-  <xacro:include filename="$(find summer_robot_description)/xacro/omni_wheel.xacro" />
-  <link name="base_footprint"/>
-  <joint name="footprint_base_joint" type="fixed">
+<robot xmlns:xacro="http://www.ros.org/wiki/xacro" name="omni_robot">
+<!-- 慣性モーメント自動計算用マクロの定義 -->
+<!-- ボックス（直方体）用 -->
+<xacro:macro name="box_inertial" params="mass x y z *origin">
+  <inertial>
+    <xacro:insert_block name="origin"/>
+    <mass value="${mass}"/>
+    <inertia ixx="${mass*(y*y+z*z)/12}" ixy="0" ixz="0"
+             iyy="${mass*(x*x+z*z)/12}" iyz="0"
+             izz="${mass*(x*x+y*y)/12}"/>
+  </inertial>
+</xacro:macro>
+<!-- シリンダ（円柱）用 -->
+<xacro:macro name="cylinder_inertial" params="mass r h *origin">
+  <inertial>
+    <xacro:insert_block name="origin"/>
+    <mass value="${mass}"/>
+    <inertia ixx="${mass*(3*r*r+h*h)/12}" ixy="0" ixz="0"
+             iyy="${mass*(3*r*r+h*h)/12}" iyz="0"
+             izz="${mass*r*r/2}"/>
+  </inertial>
+</xacro:macro>
+<xacro:property name="robot_size" value="0.7" />
+<link name="base_footprint"/>
+<link name="base_link">
+    <visual>
+        <geometry>
+            <box size="${robot_size} ${robot_size} 0.015"/>
+        </geometry>
+    </visual>
+    <collision>
+        <geometry>
+            <box size="${robot_size} ${robot_size} 0.015"/>
+        </geometry>
+    </collision>
+    <xacro:box_inertial mass="5.0" x="${robot_size}" y="${robot_size}" z="0.015">
+        <origin xyz="0 0 0" rpy="0 0 0" />
+    </xacro:box_inertial>
+</link>
+<joint name="base_joint" type="fixed">
     <parent link="base_footprint"/>
-    <child  link="base_link"/>
-    <origin xyz="0 0 0" rpy="0 0 0"/>
+    <child link="base_link"/>
+</joint>
+<xacro:macro name="wheel" params="prefix angle">
+<link name="${prefix}">
+    <visual>
+        <geometry>
+            <cylinder length="0.02" radius="0.05"/>
+        </geometry>
+    </visual>
+    <collision>
+        <geometry>
+            <cylinder length="0.02" radius="0.05"/>
+        </geometry>
+    </collision>
+    <xacro:cylinder_inertial mass="0.1" r="0.05" h="0.02">
+        <origin xyz="0 0 0" rpy="0 0 0" />
+    </xacro:cylinder_inertial>
+</link>
+<!-- オムニホイールの滑り表現用の摩擦設定 -->
+<gazebo reference="${prefix}">
+    <mu1>1.0</mu1>
+    <mu2>0.0</mu2>
+    <fdir1>1 0 0</fdir1>
+</gazebo>
+<joint name="${prefix}_joint" type="continuous">
+    <parent link="base_link"/>
+    <child link="${prefix}"/>
+    <origin rpy="${pi/2} 0 ${pi/2+angle}" xyz="${robot_size/2*1.41421356*cos(angle)} ${robot_size/2*1.41421356*sin(angle)} 0" />
+    <axis xyz="0 0 1" />
+</joint>
+<ros2_control name="${prefix}_shaft_trans" type="system">
+  <hardware>
+    <plugin>gz_ros2_control/GazeboSimSystem</plugin>
+  </hardware>
+  <joint name="${prefix}_joint">
+    <command_interface name="velocity"/>
+    <state_interface name="position" />
+    <state_interface name="velocity" />
   </joint>
-  <link name="base_link"/>
-  <joint name="laser_joint" type="fixed">
-    <parent link="base_link"/>
-    <child link="laser"/>
-    <origin xyz="0.0 0.0 0.15" rpy="0 0 0"/>
-  </joint>
-  <link name="laser">
-    <visual>
-      <origin xyz="0 0 0" rpy="0 0 0"/>
-      <geometry>
-        <cylinder length="0.04" radius="0.05"/>
-      </geometry>
-      <material name="laser_material">
-        <color rgba="0.13 0.13 0.13 1.0"/>
-      </material>
-    </visual>
-    <collision>
-      <origin xyz="0 0 0" rpy="0 0 0"/>
-      <geometry>
-        <cylinder length="0.04" radius="0.05"/>
-      </geometry>
-    </collision>
-    <inertial>
-      <origin xyz="0 0 0" rpy="0 0 0"/>
-      <mass value="0.1"/>
-      <inertia ixx="0.0001" ixy="0" ixz="0" iyy="0.0001" iyz="0" izz="0.0001"/>
-    </inertial>
-  </link>
- <gazebo reference="laser">
-  <visual>
-    <material>
-      <ambient>0.13 0.13 0.13 1.0</ambient>
-      <diffuse>0.13 0.13 0.13 1.0</diffuse>
-    </material>
-  </visual>
-  <sensor name="laser" type="gpu_lidar">
-    <pose>0 0 0 0 0 0</pose>
-    <always_on>true</always_on>
-    <visualize>true</visualize>
-    <update_rate>30</update_rate>
-    <topic>/scan</topic>
-    <lidar>
-      <scan>
-        <horizontal>
-          <samples>720</samples>
-          <resolution>1</resolution>
-          <min_angle>-3.14159</min_angle>
-          <max_angle>3.14159</max_angle>
-        </horizontal>
-      </scan>
-      <range>
-        <min>0.05</min>
-        <max>10.0</max>
-        <resolution>0.01</resolution>
-      </range>
-      <noise>
-        <type>gaussian</type>
-        <mean>0.0</mean>
-        <stddev>0.01</stddev>
-      </noise>
-    </lidar>
-  </sensor>
-  <sensor name="imu_sensor" type="imu">
-    <always_on>1</always_on>
-    <update_rate>1</update_rate>
-    <visualize>true</visualize>
-    <topic>imu</topic>
-  </sensor>
-</gazebo>
-  <joint name="body_joint" type="fixed">
-    <parent link="base_link"/>
-    <child  link="body_link"/>
-    <origin xyz="0 0 0.05" rpy="0 0 0"/>
-  </joint>
-  <link name="body_link">
-    <visual>
-      <geometry>
-        <box size="0.12 0.12 0.02" />
-      </geometry>
-      <material name="gray"/>
-    </visual>
-    <collision>
-      <geometry>
-        <box size="0.12 0.12 0.02" />
-      </geometry>
-      <surface>
-        <contact>
-          <collide_bitmask>0x01</collide_bitmask>
-        </contact>
-      </surface>
-    </collision>
-    <inertial>
-      <mass value="2.0"/>
-      <inertia ixx="0.01" ixy="0" ixz="0" iyy="0.01" iyz="0" izz="0.01"/>
-    </inertial>
-  </link>
-  <gazebo reference="body_link">
-    <visual>
-      <material>
-        <ambient>0.8 0.8 0.8 1.0</ambient>
-        <diffuse>0.8 0.8 0.8 1.0</diffuse>
-      </material>
-    </visual>
-  </gazebo>
-  <joint name="wheel0_attach_joint" type="fixed">
-    <parent link="base_link"/>
-    <child  link="wheel0_attach_link"/>
-    <origin xyz="${0.07*cos(0)} ${0.07*sin(0)} 0.019" rpy="0 0 ${0}"/>
-  </joint>
-  <link name="wheel0_attach_link" />
-  <xacro:omni_wheel_set prefix="wheel0" parent="wheel0_attach_link" />
-  <joint name="wheel1_attach_joint" type="fixed">
-    <parent link="base_link"/>
-    <child  link="wheel1_attach_link"/>
-    <origin xyz="${0.07*cos(pi/2)} ${0.07*sin(pi/2)} 0.019" rpy="0 0 ${pi/2}"/>
-  </joint>
-  <link name="wheel1_attach_link" />
-  <xacro:omni_wheel_set prefix="wheel1" parent="wheel1_attach_link" />
-  <joint name="wheel2_attach_joint" type="fixed">
-    <parent link="base_link"/>
-    <child  link="wheel2_attach_link"/>
-    <origin xyz="${0.07*cos(pi)} ${0.07*sin(pi)} 0.019" rpy="0 0 ${pi}"/>
-  </joint>
-  <link name="wheel2_attach_link" />
-  <xacro:omni_wheel_set prefix="wheel2" parent="wheel2_attach_link" />
-  <joint name="wheel3_attach_joint" type="fixed">
-    <parent link="base_link"/>
-    <child  link="wheel3_attach_link"/>
-    <origin xyz="${0.07*cos(3*pi/2)} ${0.07*sin(3*pi/2)} 0.019" rpy="0 0 ${3*pi/2}"/>
-  </joint>
-  <link name="wheel3_attach_link" />
-  <xacro:omni_wheel_set prefix="wheel3" parent="wheel3_attach_link" />
+</ros2_control>
+</xacro:macro>
+<xacro:wheel prefix="wheel0_motor_shaft" angle="${pi/4}"/>
+<xacro:wheel prefix="wheel1_motor_shaft" angle="${3*pi/4}"/>
+<xacro:wheel prefix="wheel2_motor_shaft" angle="${5*pi/4}"/>
+<xacro:wheel prefix="wheel3_motor_shaft" angle="${7*pi/4}"/>
+<link name="lidar_link">
+    <visual>
+        <geometry>
+            <cylinder length="0.05" radius="0.05"/>
+        </geometry>
+    </visual>
+    <collision>
+        <geometry>
+            <cylinder length="0.05" radius="0.05"/>
+        </geometry>
+    </collision>
+    <xacro:cylinder_inertial mass="0.1" r="0.05" h="0.05">
+        <origin xyz="0 0 0" rpy="0 0 0" />
+    </xacro:cylinder_inertial>
+</link>
+<joint name="lidar_link_joint" type="continuous">
+    <parent link="base_link"/>
+    <child link="lidar_link"/>
+    <origin rpy="0 0 0" xyz="0 0 0.02" />
+    <axis xyz="0 0 1" />
+</joint>
+<xacro:macro name="arm" params="prefix xyz rpy">
+<link name="${prefix}_base_link">
+    <visual>
+        <geometry>
+            <box size="0.1 0.1 0.5"/>
+        </geometry>
+    </visual>
+</link>
+<joint name="${prefix}_base_joint" type="fixed">
+    <parent link="base_link"/>
+    <child link="${prefix}_base_link"/>
+    <origin rpy="${rpy}" xyz="${xyz}" />
+</joint>
+<xacro:property name="arm_link_length" value="0.3" />
+<link name="${prefix}_link">
+    <visual>
+        <origin rpy="0 0 0" xyz="0 ${arm_link_length/2} 0" />
+        <geometry>
+            <box size="0.1 ${arm_link_length} 0.1"/>
+        </geometry>
+    </visual>
+    <collision>
+        <origin rpy="0 0 0" xyz="0 ${arm_link_length/2} 0" />
+        <geometry>
+            <box size="0.1 ${arm_link_length} 0.1"/>
+        </geometry>
+    </collision>
+    <xacro:box_inertial mass="0.5" x="0.1" y="${arm_link_length}" z="0.1">
+        <origin rpy="0 0 0" xyz="0 ${arm_link_length/2} 0" />
+    </xacro:box_inertial>
+</link>
+<joint name="${prefix}_joint" type="revolute">
+    <parent link="${prefix}_base_link"/>
+    <child link="${prefix}_link"/>
+    <origin rpy="0 0 0" xyz="0 0 0" />
+    <axis xyz="1 0 0" />
+    <limit effort="1000.0" lower="-0.7" upper="0.7" velocity="0.5"/>
+</joint>
+<xacro:property name="arm_link2_length" value="0.2" />
+<link name="${prefix}_link2">
+    <visual>
+        <origin rpy="0 0 0" xyz="0 ${arm_link2_length/2} 0" />
+        <geometry>
+            <box size="0.1 ${arm_link2_length} 0.1"/>
+        </geometry>
+    </visual>
+    <collision>
+        <origin rpy="0 0 0" xyz="0 ${arm_link2_length/2} 0" />
+        <geometry>
+            <box size="0.1 ${arm_link2_length} 0.1"/>
+        </geometry>
+    </collision>
+    <xacro:box_inertial mass="0.3" x="0.1" y="${arm_link2_length}" z="0.1">
+        <origin rpy="0 0 0" xyz="0 ${arm_link2_length/2} 0" />
+    </xacro:box_inertial>
+</link>
+<joint name="${prefix}_joint2" type="revolute">
+    <parent link="${prefix}_link"/>
+    <child link="${prefix}_link2"/>
+    <origin rpy="0 0 0" xyz="0 ${arm_link_length} 0" />
+    <axis xyz="1 0 0" />
+    <limit effort="1000.0" lower="-0.7" upper="0.7" velocity="0.5"/>
+</joint>
+</xacro:macro>
+<xacro:arm prefix="arm1" xyz="0 0.3 0.25" rpy="0 0 0"/>
+<xacro:arm prefix="arm2" xyz="0.2 0.3 0.25" rpy="0 0 0"/>
+<xacro:arm prefix="arm3" xyz="-0.2 0.3 0.25" rpy="0 0 0"/>
+<xacro:arm prefix="arm4" xyz="0 -0.3 0.25" rpy="0 0 ${pi}"/>
+<xacro:arm prefix="arm5" xyz="0.2 -0.3 0.25" rpy="0 0 ${pi}"/>
+<xacro:arm prefix="arm6" xyz="-0.2 -0.3 0.25" rpy="0 0 ${pi}"/>
+<link name="camera_link">
+    <visual>
+        <geometry>
+            <box size="0.1 0.1 0.1"/>
+        </geometry>
+    </visual>
+</link>
+<joint name="camera_joint" type="fixed">
+    <parent link="base_link"/>
+    <child link="camera_link"/>
+    <origin rpy="${-pi/4} 0 0" xyz="0 0.3 0.75" />
+</joint>
+<link name="camera_link2">
+    <visual>
+        <geometry>
+            <box size="0.1 0.1 0.1"/>
+        </geometry>
+    </visual>
+</link>
+<joint name="camera_joint2" type="fixed">
+    <parent link="base_link"/>
+    <child link="camera_link2"/>
+    <origin rpy="${-pi/4} 0 ${pi}" xyz="0 -0.3 0.75" />
+</joint>
+<xacro:macro name="gather" params="prefix xyz">
+<link name="${prefix}_base_link">
+    <visual>
+        <geometry>
+            <box size="0.1 0.1 0.5"/>
+        </geometry>
+    </visual>
+</link>
+<joint name="${prefix}_base_joint" type="fixed">
+    <parent link="base_link"/>
+    <child link="${prefix}_base_link"/>
+    <origin rpy="0 0 0" xyz="${xyz}" />
+</joint>
+<link name="${prefix}_link">
+    <visual>
+        <geometry>
+            <box size="0.3 0.1 0.1"/>
+        </geometry>
+    </visual>
+    <collision>
+        <geometry>
+            <box size="0.3 0.1 0.1"/>
+        </geometry>
+    </collision>
+    <xacro:box_inertial mass="0.3" x="0.3" y="0.1" z="0.1">
+        <origin xyz="0 0 0" rpy="0 0 0" />
+    </xacro:box_inertial>
+</link>
+<joint name="${prefix}_joint" type="prismatic">
+    <parent link="${prefix}_base_link"/>
+    <child link="${prefix}_link"/>
+    <origin rpy="0 0 0" xyz="0.2 0 0" />
+    <axis xyz="0 0 1" />
+    <limit effort="1000.0" lower="-0.2" upper="0.2" velocity="0.5"/>
+</joint>
+</xacro:macro>
+<xacro:gather prefix="gather1" xyz="0.3 0.1 0.25"/>
+<xacro:gather prefix="gather2" xyz="0.3 -0.1 0.25"/>
+<link name="camera_link3">
+    <visual>
+        <geometry>
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