Commit message: gazeboを軽くするための変更

File: summer_robot_description/xacro/omni_wheel.xacro (robot description, xacro)
@@ -1,6 +1,6 @@
+<?xml version="1.0"?>
 <robot xmlns:xacro="http://ros.org/wiki/xacro">
-  <!--コロの定義-->
   <xacro:macro name="barrel" params="prefix parent dir">
-    <joint name="${prefix}_joint" type="continuous"><!-- continuous -->
+    <joint name="${prefix}_joint" type="continuous">
       <parent link="${parent}"/>
       <child link="${prefix}_link"/>
@@ -9,14 +9,4 @@
       <dynamics damping="0.001"/>
     </joint>
-    <!--<ros2_control name="${prefix}_trans" type="system">
-      <hardware>
-        <plugin>gz_ros2_control/GazeboSimSystem</plugin>
-      </hardware>
-      <joint name="${prefix}_joint">
-        <command_interface name="effort" />
-        <state_interface name="position" />
-        <state_interface name="velocity" />
-      </joint>
-    </ros2_control>-->
     <link name="${prefix}_link">
       <visual>
@@ -24,18 +14,19 @@
           <mesh filename="package://summer_robot_description/meshes/omni_barrel.stl" />
         </geometry>
-        <material name="black"/>
+        <material name="black">
+          <color rgba="0.1 0.1 0.1 1.0"/>
+        </material>
       </visual>
-      <!--<collision>
-        <geometry>
-          <mesh filename="package://summer_robot_description/meshes/omni_barrel.stl" />
-        </geometry>
-      </collision>-->
-       <collision>
-        <!-- STLをやめてcylinderに変更 -->
+      <collision>
         <origin rpy="0 0 0" xyz="0 0 0"/>
         <geometry>
-            <cylinder radius="0.007" length="0.012"/>
+          <cylinder radius="0.007" length="0.012"/>
         </geometry>
-    </collision>
+        <surface>
+          <contact>
+            <collide_bitmask>0x01</collide_bitmask>
+          </contact>
+        </surface>
+      </collision>
       <inertial>
         <mass value="0.002"/>
@@ -48,28 +39,12 @@
       <kp value="5000" />
       <kd value="10" />
-      <material>Gazebo/Black</material>
-    </gazebo>
-    <!--コロに謎の白い箱を追加している-->
-    <joint name="${prefix}_mark_joint" type="fixed">
-      <parent link="${prefix}_link"/>
-      <child link="${prefix}_mark_link"/>
-      <origin rpy="0 0 0" xyz="0.005 0 0"/>
-    </joint>
-    <link name="${prefix}_mark_link">
       <visual>
-        <geometry>
-          <box size="0.005 0.005 0.005"/>
-        </geometry>
-        <material name="white"/>
+        <material>
+          <ambient>0.2 0.2 0.2 1.0</ambient>
+          <diffuse>0.2 0.2 0.2 1.0</diffuse>
+        </material>
       </visual>
-    </link>
-    <gazebo reference="${prefix}_mark_link">
-      <material>Gazebo/White</material>
     </gazebo>
   </xacro:macro>
-  <!--モータ(可動部)の定義-->
-  <!--
-  [${parent}]->(${prefix}_joint)->[${prefix}_body_link {モータのstl}]->(${prefix}_shaft_joint {モータ（可動部）} )->[${prefix}_shaft_link {軸のstl}]
-  -->
   <xacro:macro name="motor" params="prefix parent">
     <joint name="${prefix}_joint" type="fixed">
@@ -78,5 +53,4 @@
       <origin xyz="0 0 0" rpy="0 0 0"/>
     </joint>
-    <!--モータ-->
     <link name="${prefix}_body_link">
       <visual>
@@ -84,5 +58,7 @@
           <mesh filename="package://summer_robot_description/meshes/ga25_body.stl" />
         </geometry>
-        <material name="gray"/>
+        <material name="gray">
+          <color rgba="0.5 0.5 0.5 1.0"/>
+        </material>
       </visual>
       <collision>
@@ -91,4 +67,9 @@
           <cylinder radius="0.012" length="0.05" />
         </geometry>
+        <surface>
+          <contact>
+            <collide_bitmask>0x01</collide_bitmask>
+          </contact>
+        </surface>
       </collision>
       <inertial>
@@ -98,5 +79,10 @@
     </link>
     <gazebo reference="${prefix}_body_link">
-      <material>Gazebo/Gray</material>
+      <visual>
+        <material>
+          <ambient>0.5 0.5 0.5 1.0</ambient>
+          <diffuse>0.5 0.5 0.5 1.0</diffuse>
+        </material>
+      </visual>
     </gazebo>
     <joint name="${prefix}_shaft_joint" type="continuous">
@@ -118,5 +104,4 @@
       </joint>
     </ros2_control>
-    <!--軸-->
     <link name="${prefix}_shaft_link">
       <visual>
@@ -124,5 +109,7 @@
           <mesh filename="package://summer_robot_description/meshes/ga25_shaft.stl" />
         </geometry>
-        <material name="gray"/>
+        <material name="gray">
+          <color rgba="0.5 0.5 0.5 1.0"/>
+        </material>
       </visual>
       <inertial>
@@ -132,8 +119,13 @@
     </link>
     <gazebo reference="${prefix}_shaft_link">
-      <material>Gazebo/Gray</material>
+      <self_collide>false</self_collide>
+      <visual>
+        <material>
+          <ambient>0.5 0.5 0.5 1.0</ambient>
+          <diffuse>0.5 0.5 0.5 1.0</diffuse>
+        </material>
+      </visual>
     </gazebo>
   </xacro:macro>
-  <!--全体の組み合わせ-->
   <xacro:macro name="omni_wheel_set" params="prefix parent">
     <joint name="${prefix}_base_joint" type="fixed">
@@ -155,6 +147,19 @@
         </geometry>
         <origin xyz="0 0 0" rpy="0 0 0"/>
-        <material name="gray"/>
+        <material name="gray">
+          <color rgba="0.5 0.5 0.5 1.0"/>
+        </material>
       </visual>
+      <collision>
+        <origin rpy="0 0 0" xyz="0 0 0"/>
+        <geometry>
+          <cylinder radius="0.03" length="0.02" />
+        </geometry>
+        <surface>
+          <contact>
+            <collide_bitmask>0x01</collide_bitmask>
+          </contact>
+        </surface>
+      </collision>
       <inertial>
         <mass value="0.025"/>
@@ -163,5 +168,10 @@
     </link>
     <gazebo reference="${prefix}_housing_link">
-      <material>Gazebo/Gray</material>
+      <visual>
+        <material>
+          <ambient>0.5 0.5 0.5 1.0</ambient>
+          <diffuse>0.5 0.5 0.5 1.0</diffuse>
+        </material>
+      </visual>
     </gazebo>
     <joint name="${prefix}_housing_s_joint" type="fixed">

File: summer_robot_description/xacro/robot.xacro (robot description, xacro)
@@ -1,23 +1,24 @@
+<?xml version="1.0"?>
 <robot xmlns:xacro="http://ros.org/wiki/xacro" name="my_omni_robot">
-    <material name="gray">
-      <color rgba="0.8 0.8 0.8 1.0"/>
-    </material>
-    <material name="black">
-      <color rgba="0 0 0 1.0"/>
-    </material>
-    <material name="white">
-      <color rgba="1.0 1.0 1.0 1.0"/>
-    </material>
-    <material name="red">
-      <color rgba="1.0 0 0 1.0"/>
-    </material>
-    <material name="light_red">
-      <color rgba="1.0 0.5 0.5 1.0"/>
-    </material>
-    <material name="yellow">
-      <color rgba="0 1.0 1.0 1.0"/>
-    </material>
-    <xacro:include filename="$(find summer_robot_description)/xacro/omni_wheel.xacro" />
-    <link name="base_footprint"/>
+  <material name="gray">
+    <color rgba="0.8 0.8 0.8 1.0"/>
+  </material>
+  <material name="black">
+    <color rgba="0 0 0 1.0"/>
+  </material>
+  <material name="white">
+    <color rgba="1.0 1.0 1.0 1.0"/>
+  </material>
+  <material name="red">
+    <color rgba="1.0 0 0 1.0"/>
+  </material>
+  <material name="light_red">
+    <color rgba="1.0 0.5 0.5 1.0"/>
+  </material>
+  <material name="yellow">
+    <color rgba="0 1.0 1.0 1.0"/>
+  </material>
+  <xacro:include filename="$(find summer_robot_description)/xacro/omni_wheel.xacro" />
+  <link name="base_footprint"/>
   <joint name="footprint_base_joint" type="fixed">
     <parent link="base_footprint"/>
@@ -25,71 +26,72 @@
     <origin xyz="0 0 0" rpy="0 0 0"/>
   </joint>
-   <link name="base_link"/>
-   <!-- ========== LiDAR Joint ========== -->
-<joint name="laser_joint" type="fixed">
+  <link name="base_link"/>
+  <joint name="laser_joint" type="fixed">
     <parent link="base_link"/>
     <child link="laser"/>
     <origin xyz="0.0 0.0 0.15" rpy="0 0 0"/>
-</joint>
-<!-- ========== LiDAR Link ========== -->
-<link name="laser">
+  </joint>
+  <link name="laser">
     <visual>
-        <origin xyz="0 0 0" rpy="0 0 0"/>
-        <geometry>
-            <cylinder length="0.04" radius="0.05"/>
-        </geometry>
-        <material name="laser_material">
-            <color rgba="0.13 0.13 0.13 1.0"/>
-        </material>
+      <origin xyz="0 0 0" rpy="0 0 0"/>
+      <geometry>
+        <cylinder length="0.04" radius="0.05"/>
+      </geometry>
+      <material name="laser_material">
+        <color rgba="0.13 0.13 0.13 1.0"/>
+      </material>
     </visual>
     <collision>
-        <origin xyz="0 0 0" rpy="0 0 0"/>
-        <geometry>
-            <cylinder length="0.04" radius="0.05"/>
-        </geometry>
+      <origin xyz="0 0 0" rpy="0 0 0"/>
+      <geometry>
+        <cylinder length="0.04" radius="0.05"/>
+      </geometry>
     </collision>
     <inertial>
-        <origin xyz="0 0 0" rpy="0 0 0"/>
-        <mass value="0.1"/>
-        <inertia ixx="0.0001" ixy="0" ixz="0"
-                 iyy="0.0001" iyz="0" izz="0.0001"/>
+      <origin xyz="0 0 0" rpy="0 0 0"/>
+      <mass value="0.1"/>
+      <inertia ixx="0.0001" ixy="0" ixz="0" iyy="0.0001" iyz="0" izz="0.0001"/>
     </inertial>
-</link>
-<!-- ========== Gazebo Sensor ========== -->
-<gazebo reference="laser">
-    <sensor name="laser" type="gpu_lidar">
-        <pose>0 0 0 0 0 0</pose>
-        <always_on>true</always_on>
-        <visualize>true</visualize>
-        <update_rate>30</update_rate>
-        <topic>/scan</topic>
-        <gz_frame_id>laser</gz_frame_id>
-        <lidar>
-            <scan>
-                <horizontal>
-                    <samples>720</samples>
-                    <resolution>1</resolution>
-                    <min_angle>-3.14159</min_angle>
-                    <max_angle>3.14159</max_angle>
-                </horizontal>
-            </scan>
-            <range>
-                <min>0.05</min>
-                <max>10.0</max>
-                <resolution>0.01</resolution>
-            </range>
-            <noise>
-                <type>gaussian</type>
-                <mean>0.0</mean>
-                <stddev>0.01</stddev>
-            </noise>
-        </lidar>
-    </sensor>
-    <sensor name="imu_sensor" type="imu">
-      <always_on>1</always_on>
-      <update_rate>1</update_rate>
-      <visualize>true</visualize>
+  </link>
+ <gazebo reference="laser">
+  <visual>
+    <material>
+      <ambient>0.13 0.13 0.13 1.0</ambient>
+      <diffuse>0.13 0.13 0.13 1.0</diffuse>
+    </material>
+  </visual>
+  <sensor name="laser" type="gpu_lidar">
+    <pose>0 0 0 0 0 0</pose>
+    <always_on>true</always_on>
+    <visualize>true</visualize>
+    <update_rate>30</update_rate>
+    <topic>/scan</topic>
+    <lidar>
+      <scan>
+        <horizontal>
+          <samples>720</samples>
+          <resolution>1</resolution>
+          <min_angle>-3.14159</min_angle>
+          <max_angle>3.14159</max_angle>
+        </horizontal>
+      </scan>
+      <range>
+        <min>0.05</min>
+        <max>10.0</max>
+        <resolution>0.01</resolution>
+      </range>
+      <noise>
+        <type>gaussian</type>
+        <mean>0.0</mean>
+        <stddev>0.01</stddev>
+      </noise>
+    </lidar>
+  </sensor>
+  <sensor name="imu_sensor" type="imu">
+    <always_on>1</always_on>
+    <update_rate>1</update_rate>
+    <visualize>true</visualize>
     <topic>imu</topic>
-</sensor>
+  </sensor>
 </gazebo>
   <joint name="body_joint" type="fixed">
@@ -109,4 +111,9 @@
         <box size="0.12 0.12 0.02" />
       </geometry>
+      <surface>
+        <contact>
+          <collide_bitmask>0x01</collide_bitmask>
+        </contact>
+      </surface>
     </collision>
     <inertial>
@@ -115,4 +122,12 @@
     </inertial>
   </link>
+  <gazebo reference="body_link">
+    <visual>
+      <material>
+        <ambient>0.8 0.8 0.8 1.0</ambient>
+        <diffuse>0.8 0.8 0.8 1.0</diffuse>
+      </material>
+    </visual>
+  </gazebo>
   <joint name="wheel0_attach_joint" type="fixed">
     <parent link="base_link"/>

File: summer_robot_field_description/urdf/field.urdf (robot description, URDF)
Before this commit: robot my_field, 1 links, 0 joints
Links:
- link field_link: geometry collision box size=3.5 7.0 0.001; visual mesh filename=package://summer_robot_field_description/meshes/summer_robo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
